Commit message: 修改urdf

File: src/machine/urdf/turtlebot_properties.urdf.xacro (robot description, xacro)
@@ -19,7 +19,9 @@
      (currently in development and awaiting feedback)
    -->
-	<xacro:property name="cam_px" value="-0.087" />
+	<!--<xacro:property name="cam_px" value="-0.087" />-->
 <!--	<xacro:property name="cam_py" value="-0.0125" /> Y varies for different configurations. get sets in sensors_urdf -->
-	<xacro:property name="cam_pz" value="0.2870" />
+	<!--<xacro:property name="cam_pz" value="0.2870" />-->
+	<xacro:property name="cam_px" value="0.13" />
+	<xacro:property name="cam_pz" value="0.87" />
 	<xacro:property name="cam_or" value="0" />
 	<xacro:property name="cam_op" value="0" />
