Commit message: 修改了amcl参数，添加了camera odom，task修改了follow的plan添加了keyboardcontrol的速度调节，添加了简易版本的gotask，basecontrol添加了预先产生一个控制向量功能obstaclewarning修改投影机制，readmap修改了障碍物记忆功能

File: src/machine/urdf/sensors/asus_xtion_pro.urdf.xacro (robot description, xacro)
@@ -66,5 +66,5 @@
     <!-- Asus mount -->
     <joint name="mount_asus_xtion_pro_joint" type="fixed">
-      <origin xyz="-0.1024 0.0 0.272" rpy="0 0 0"/>
+      <origin xyz="0.1024 0.0 0.85" rpy="0 0 0"/>
       <parent link="${parent}"/>
       <child link="mount_asus_xtion_pro_link"/>
